Commit message: Update tita_description.urdf
change the torque limit from 45 to 60

Signed-off-by: yankai <1924286463@qq.com>

File: resources/tita/urdf/tita_description.urdf (robot description, URDF)
Before this commit: robot tita_ros2_control, 14 links, 13 joints
Joints:
- joint joint_left_leg_1: limit lower=-0.785398 upper=0.785398 effort=45 velocity=25 -> lower=-0.785398 upper=0.785398 effort=60 velocity=25
- joint joint_left_leg_2: limit lower=-1.919862 upper=3.490659 effort=45 velocity=25 -> lower=-1.919862 upper=3.490659 effort=60 velocity=25
- joint joint_left_leg_3: limit lower=-2.670354 upper=-0.698132 effort=45 velocity=25 -> lower=-2.670354 upper=-0.698132 effort=60 velocity=25
- joint joint_right_leg_1: limit lower=-0.785398 upper=0.785398 effort=45 velocity=25 -> lower=-0.785398 upper=0.785398 effort=60 velocity=25
- joint joint_right_leg_2: limit lower=-1.919862 upper=3.490659 effort=45 velocity=25 -> lower=-1.919862 upper=3.490659 effort=60 velocity=25
- joint joint_right_leg_3: limit lower=-2.670354 upper=-0.698132 effort=45 velocity=25 -> lower=-2.670354 upper=-0.698132 effort=60 velocity=25

Commit message: uv setup and wheel changes

File: resources/tita/urdf/tita_description.urdf (robot description, URDF)
Before this commit: robot tita_ros2_control, 14 links, 13 joints
Links:
- added link left_leg_4_1, mass 1.5094; collision cylinder length=0.034 radius=0.04625; visual mesh filename=../meshes/left_leg_4.STL scale=0.5 0.5 1
- added link left_leg_4_3, mass 1.5094; collision cylinder length=0.034 radius=0.04625; visual mesh filename=../meshes/left_leg_4.STL scale=0.5 0.5 1
- added link left_leg_4_bar, mass 0.1; collision box size=0.05 0.215 0.005; visual box size=0.05 0.215 0.005
- added link right_leg_4_1, mass 1.5094; collision cylinder length=0.034 radius=0.04625; visual mesh filename=../meshes/right_leg_4.STL scale=0.5 0.5 1
- added link right_leg_4_3, mass 1.5094; collision cylinder length=0.034 radius=0.04625; visual mesh filename=../meshes/right_leg_4.STL scale=0.5 0.5 1
- added link right_leg_4_bar, mass 0.1; collision box size=0.05 0.215 0.005; visual box size=0.05 0.215 0.005
- link left_leg_4: geometry collision cylinder length=0.034 radius=0.04625; visual mesh filename=../meshes/left_leg_4.STL scale=0.5 0.5 1
- link right_leg_4: geometry collision cylinder length=0.034 radius=0.04625; visual mesh filename=../meshes/right_leg_4.STL scale=0.5 0.5 1
Joints:
- added joint joint_left_leg_4_1: type revolute, parent left_leg_4_bar, child left_leg_4_1, origin xyz=0 -0.095 0.0205 rpy=0 0 0, axis 0 0 1, limit lower=-999999 upper=999999 effort=15 velocity=20
- added joint joint_left_leg_4_3: type revolute, parent left_leg_4_bar, child left_leg_4_3, origin xyz=0 0.095 0.0205 rpy=0 0 0, axis 0 0 1, limit lower=-999999 upper=999999 effort=15 velocity=20
- added joint joint_left_leg_4_bar: type revolute, parent left_leg_3, child left_leg_4_bar, origin xyz=0.2 0 0.03 rpy=0 0 0.75, axis 0 0 1, limit lower=-0.785398 upper=0.785398 effort=45 velocity=25
- added joint joint_right_leg_4_1: type revolute, parent right_leg_4_bar, child right_leg_4_1, origin xyz=0 -0.095 -0.0205 rpy=0 0 0, axis 0 0 1, limit lower=-999999 upper=999999 effort=15 velocity=20
- added joint joint_right_leg_4_3: type revolute, parent right_leg_4_bar, child right_leg_4_3, origin xyz=0 0.095 -0.0205 rpy=0 0 0, axis 0 0 1, limit lower=-999999 upper=999999 effort=15 velocity=20
- added joint joint_right_leg_4_bar: type revolute, parent right_leg_3, child right_leg_4_bar, origin xyz=0.2 0 -0.03 rpy=0 0 0.75, axis 0 0 1, limit lower=-0.785398 upper=0.785398 effort=45 velocity=25
- joint joint_left_leg_1: limit lower=-0.785398 upper=0.785398 effort=60 velocity=25 -> lower=-0.785398 upper=0.785398 effort=45 velocity=25
- joint joint_left_leg_2: limit lower=-1.919862 upper=3.490659 effort=60 velocity=25 -> lower=-1.919862 upper=3.490659 effort=45 velocity=25
- joint joint_left_leg_3: limit lower=-2.670354 upper=-0.698132 effort=60 velocity=25 -> lower=-2.670354 upper=-0.698132 effort=45 velocity=25
- joint joint_left_leg_4: origin xyz=0.2 0 0.0514 rpy=0 0 0 -> xyz=0 0 0.0205 rpy=0 0 0; parent left_leg_3 -> left_leg_4_bar
- joint joint_right_leg_1: limit lower=-0.785398 upper=0.785398 effort=60 velocity=25 -> lower=-0.785398 upper=0.785398 effort=45 velocity=25
- joint joint_right_leg_2: limit lower=-1.919862 upper=3.490659 effort=60 velocity=25 -> lower=-1.919862 upper=3.490659 effort=45 velocity=25
- joint joint_right_leg_3: limit lower=-2.670354 upper=-0.698132 effort=60 velocity=25 -> lower=-2.670354 upper=-0.698132 effort=45 velocity=25
- joint joint_right_leg_4: origin xyz=0.2 0 -0.0514 rpy=0 0 0 -> xyz=0 0 -0.0205 rpy=0 0 0; parent right_leg_3 -> right_leg_4_bar
